Commit message: Refactor/shared/wheel odom fix (#590)
* fix in sim_gz.launch.py

* fix urdf rover model (rockers and wheels)

* fix wheels odometry

* partially fix

* feature: add parameter to remove stereo camera from urdf and rviz visualization

* fix: add processing motors' encoders to absolute position

* change shape of wheels to make odometry behaviour more deterministic

File: src/rover_description/urdf/macros/wheel_assembly.xacro (robot description, xacro)
@@ -11,5 +11,5 @@
       </inertial>
       <visual>
-        <origin xyz="0 ${wheel_mount_hub_offset * y_sign} ${wheel_mount_visual_z}" rpy="0 0 0"/>
+        <origin xyz="0.001 ${wheel_mount_hub_offset * y_sign} ${wheel_mount_visual_z}" rpy="0 0 0"/>
         <geometry>
           <mesh filename="package://rover_description/meshes/suspension/wheel_mount.stl" scale="1 ${y_sign} 1"/>
@@ -28,5 +28,5 @@
       <parent link="${parent}"/>
       <child link="${prefix}_wheel_mount_link"/>
-      <origin xyz="${x_sign * (rocker_length / 2.0 - rocker_mount_x_offset)} ${rocker_hub_y} ${rocker_hub_z}" rpy="0 0 0"/>
+      <origin xyz="${x_sign * (rocker_length / 2.0 - rocker_mount_x_offset)} ${rocker_hub_y * y_sign} ${rocker_hub_z}" rpy="0 0 0"/>
       <axis xyz="0 0 1"/>
       <limit lower="${-steering_limit}" upper="${steering_limit}" effort="${steering_effort}" velocity="${steering_velocity}"/>
@@ -41,14 +41,21 @@
       </inertial>
       <visual>
-        <origin xyz="0 ${wheel_hub_offset * y_sign} 0" rpy="0 0 0"/>
+        <!-- Right wheel is yawed 180 deg rather than scaled by -1: a negative
+             scale flips polygon winding, inverting the mesh normals. -->
+        <origin xyz="0 ${wheel_hub_offset * y_sign} 0" rpy="0 0 ${0 if y_sign > 0 else pi}"/>
         <geometry>
-          <mesh filename="package://rover_description/meshes/suspension/wheel.stl" scale="1 ${y_sign} 1"/>
+          <mesh filename="package://rover_description/meshes/suspension/wheel.stl" scale="1 1 1"/>
         </geometry>
         <material name="dark_wheel"/>
       </visual>
+      <!-- Sphere, not a cylinder: a flat cylinder touches the ground at one rim
+           edge in DART, which shortens the spin lever arm by wheel_width/2 and
+           made the sim rotate ~13% faster than the wheel kinematics. A sphere
+           always contacts directly under the wheel centre, at the same rolling
+           radius, and is the most stable shape against the terrain mesh. -->
       <collision>
-        <origin xyz="0 0 0" rpy="${pi / 2.0 * y_sign} 0 0"/>
+        <origin xyz="0 0 0" rpy="0 0 0"/>
         <geometry>
-          <cylinder radius="${wheel_radius}" length="${wheel_width}"/>
+          <sphere radius="${wheel_radius}"/>
         </geometry>
       </collision>

File: src/rover_description/urdf/properties.xacro (robot description, xacro)
@@ -23,10 +23,15 @@
   <xacro:property name="rocker_height" value="0.187"/>  <!-- Z -->
   <xacro:property name="rocker_mass" value="1.0"/>
-  <!-- Mesh alignment: centers rocker.stl on the rocker link's own origin -->
-  <xacro:property name="rocker_mesh_align_xyz" value="0 0.0001 0.0"/>
+  <!-- Mesh alignment: centers rocker.stl on the rocker link's own origin. The left
+       rocker's mesh is yawed 180 deg, so its Y correction is not a mirror of the right. -->
+  <xacro:property name="rocker_mesh_align_y_left" value="-0.02"/>
+  <xacro:property name="rocker_mesh_align_y_right" value="0.02"/>
   <!-- Wheel-mount attachment point: where the wheel_mount hub attaches to the rocker's end,
        relative to the rocker's pivot origin -->
+  <!-- Lateral offset stays 0: the steering axis and wheel centre sit on the rocker
+       pivot plane, so wheel centres land at +/-track_width/2, which is what
+       swerve_kinematics and the odometry in controllers.yaml assume. -->
   <xacro:property name="rocker_mount_x_offset" value="0.050"/>
-  <xacro:property name="rocker_hub_y" value="-0.0258"/>
+  <xacro:property name="rocker_hub_y" value="0.0"/>
   <xacro:property name="rocker_hub_z" value="-0.1140"/>
   <!-- ===================== WHEEL MOUNT (steering knuckle) ===================== -->
@@ -37,9 +42,9 @@
   <xacro:property name="wheel_mount_mass" value="0.162"/>
   <!-- Mesh alignment: centers wheel_mount.stl's steering bore on the link's own origin -->
-  <xacro:property name="wheel_mount_hub_offset" value="0.1253"/>
-  <xacro:property name="wheel_mount_visual_z" value="-0.1814"/>
+  <xacro:property name="wheel_mount_hub_offset" value="0.1489"/>
+  <xacro:property name="wheel_mount_visual_z" value="-0.1799"/>
   <!-- Wheel attachment point: axle position relative to the steering bore -->
   <xacro:property name="wheel_mount_drop" value="0.1857"/>
-  <xacro:property name="axle_lateral_offset" value="-0.0168"/>
+  <xacro:property name="axle_lateral_offset" value="0.0"/>
   <!-- ===================== WHEEL ===================== -->
   <!-- Geometry -->
@@ -66,6 +71,6 @@
   <xacro:property name="drive_velocity" value="10"/>
   <!-- ===================== WHEEL GROUND CONTACT FRICTION ===================== -->
-  <xacro:property name="wheel_mu1" value="1.0"/>
-  <xacro:property name="wheel_mu2" value="1.0"/>
+  <xacro:property name="wheel_mu1" value="1.2"/>
+  <xacro:property name="wheel_mu2" value="1.2"/>
   <xacro:property name="wheel_kp" value="1000000.0"/>
   <xacro:property name="wheel_kd" value="1.0"/>
